File: PCB/Board_1/Board_1.kicad_pcb (KiCad board)
At the start: 2 copper layers, 35 parts, among them J1 3.3_Direct, J10 AVR-ISP-10, J11 PWR, J2 FTDI, J3 105450-0101, J4 I/O_TEST, J5 GND_test, J6 I/0 L, J7 5V_Direct, J8 I/O H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

Commit message: PCB first board ready/Debugging UART
Parts:
- added C10: 20pf, Capacitor_SMD:C_0603_1608Metric, F.Cu at (236.5, 93.8)
- added C11: 1n, Capacitor_SMD:C_0603_1608Metric, F.Cu at (182.5, 106.2)
- added C9: 20pf, Capacitor_SMD:C_0603_1608Metric, F.Cu at (236.5, 107.9)
- added R10: 5k, Resistor_SMD:R_0603_1608Metric, F.Cu at (233.0, 117.2)
- added R11: 5k, Resistor_SMD:R_0603_1608Metric, F.Cu at (224.8, 117.2)
- added R12: 5k, Resistor_SMD:R_0603_1608Metric, F.Cu at (228.9, 117.2)
- added R13: 0, Resistor_SMD:R_0603_1608Metric, F.Cu at (190.9, 120.8)
- added R14: 0, Resistor_SMD:R_0603_1608Metric, F.Cu at (187.2, 120.8)
- added R15: 1M, Resistor_SMD:R_0603_1608Metric, F.Cu at (231.0, 101.0)
- added R16: 5k, Resistor_SMD:R_0603_1608Metric, F.Cu at (185.0, 110.8)
- added R6: 5k, Resistor_SMD:R_0603_1608Metric, F.Cu at (185.8, 100.4)
- added R7: 5k, Resistor_SMD:R_0603_1608Metric, F.Cu at (181.6, 100.4)
- added R8: 5k, Resistor_SMD:R_0603_1608Metric, F.Cu at (198.8, 100.4)
- added R9: 5k, Resistor_SMD:R_0603_1608Metric, F.Cu at (203.0, 100.4)
- added SW1: EN, Button_Switch_THT:SW_PUSH_6mm, F.Cu at (139.1, 119.6)
- added SW2: ID0, Button_Switch_THT:SW_PUSH_6mm, F.Cu at (139.1, 109.1)
- added Y1: ECS-160-20-3X-TR, 16 MHz Crystal:XTAL_ECS-160-20-3X-TR, F.Cu at (237.3, 101.1)
- TP1, TP4: value TestPoint_Flag -> TEST_TX; footprint TestPoint:TestPoint_Pad_4.0x4.0mm -> Connector_PinHeader_2.54mm:PinHeader_1x01_P2.54mm_Vertical
- TP2: footprint TestPoint:TestPoint_Pad_4.0x4.0mm -> Connector_PinHeader_2.54mm:PinHeader_1x01_P2.54mm_Vertical
- TP3: value TestPoint_Flag -> TEST_RX; footprint TestPoint:TestPoint_Pad_4.0x4.0mm -> Connector_PinHeader_2.54mm:PinHeader_1x01_P2.54mm_Vertical
- TP5: value TestPoint_Flag -> TEST_5V; footprint TestPoint:TestPoint_Pad_4.0x4.0mm -> Connector_PinHeader_2.54mm:PinHeader_1x01_P2.54mm_Vertical
- TP6: value TestPoint_Flag -> TEST_3.3V; footprint TestPoint:TestPoint_Pad_4.0x4.0mm -> Connector_PinHeader_2.54mm:PinHeader_1x01_P2.54mm_Vertical
- moved J10 85.1 mm to (237.3, 120.4)
- moved J6 82.1 mm to (239.3, 86.2), turned to 270 degrees
- moved J9 72.4 mm to (227.2, 135.3), turned to 90 degrees
- moved J8 69.9 mm to (217.8, 86.2), turned to 270 degrees
- moved J11 69.5 mm to (204.8, 135.3), turned to 90 degrees
- moved C5 61.5 mm to (232.2, 108.0), turned to 180 degrees
- moved F1 55.4 mm to (171.7, 90.9)
- moved J7 54.4 mm to (239.8, 114.1)
- moved C6 52.6 mm to (232.0, 112.4), turned to 180 degrees
- moved U4 51.5 mm to (217.1, 111.1), turned to 180 degrees
- moved C1 51.3 mm to (148.8, 124.5)
- moved J2 46.3 mm to (174.6, 135.0), turned to 90 degrees
- moved J4 46.0 mm to (155.9, 135.1), turned to 90 degrees
- moved J1 45.0 mm to (149.6, 135.1), turned to 90 degrees
- moved TP5 44.4 mm to (139.7, 86.9), turned to 180 degrees
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Connections:
- net Net-(J4-Pad1) renamed IO0
- net Net-(J6-Pad3) renamed PD2
- net Net-(J6-Pad4) renamed PD3
- net Net-(J6-Pad5) renamed PD4
- net Net-(J6-Pad6) renamed PD5
- net Net-(J6-Pad7) renamed PD6
- net Net-(J6-Pad8) renamed PD7
- net Net-(J8-Pad1) renamed PB0
- net Net-(J8-Pad2) renamed PB1
- net Net-(J8-Pad3) renamed PB2
- net Net-(J9-Pad1) renamed PC0
- net Net-(J9-Pad2) renamed PC1
- net Net-(J9-Pad3) renamed PC2
- net Net-(J9-Pad4) renamed PC3
- J4 pad 2: I034 -> IO34
- J4 pad 4: IO32 -> I032
- J4 pad 5: IO33 -> I033
- U2 pad 10: Net-(U2-Pad10) -> OE
- U2 pad 11: Net-(U2-Pad11) -> GND
- U4 pad 7: Net-(U4-Pad7) -> PB6
- U4 pad 8: Net-(U4-Pad8) -> PB7
Routing:
- net GND: track 0.00 -> 217.5 mm, vias 0 -> 23
- net +5V: track 0.00 -> 212.6 mm, vias 0 -> 6
- net +3V3: track 0.00 -> 205.5 mm, vias 0 -> 2
- net Net-(J6-Pad1): track 0.00 -> 130.3 mm, vias 0 -> 6
- net Net-(J6-Pad2): track 0.00 -> 127.1 mm, vias 0 -> 6
- net Net-(J2-Pad3): track 0.00 -> 102.1 mm, vias 0 -> 2
- net IO0: track 0.00 -> 90.3 mm, vias 0 -> 2
- net SCL: track 0.00 -> 89.0 mm, vias 0 -> 2
- net Net-(J2-Pad2): track 0.00 -> 86.1 mm, vias 0 -> 4
- net SDA: track 0.00 -> 84.5 mm, vias 0 -> 2
- net PD2: track 0.00 -> 69.4 mm, vias 0 -> 2
- net Net-(J10-Pad9): track 0.00 -> 69.3 mm, vias 0 -> 4
- net Net-(J10-Pad1): track 0.00 -> 66.4 mm, vias 0 -> 6
- net Net-(J10-Pad7): track 0.00 -> 63.7 mm, vias 0 -> 2
- net RESET: track 0.00 -> 57.6 mm, vias 0 -> 2
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- added copper zone on B.Cu, net GND
Other:
- board outline added: 108.7 x 58.4 mm
- net class Default: clearance 0.2 -> 0.1524; trace_width 0.25 -> 0.1524; via_dia 0.8 -> 0.6858; via_drill 0.4 -> 0.3302
- rule solder_mask_min_width: 0.25 -> 0.101
- rule trace_clearance: 0.2 -> 0.1524
- rule trace_min: 0.2 -> 0.1524
- rule via_min_size: 0.4 -> 0.508
- board text added: "SoundZue$"
