File: PCB/Board_1/Board_1.sch (KiCad schematic (older format))
At the start: 36 parts, among them J1 3.3_Direct, J2 FTDI, J3 USB_C_Receptacle_USB2.0, J4 I/0 L, J5 5V_Direct, J6 I/O H, J7 AD, J8 AVR-ISP-10, J9 PWR, U1 ESP32-WROOM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

Commit message: PCB Schematic & Footprint match Done
Parts:
- removed J3: USB_C_Receptacle_USB2.0, symbol Connector:USB_C_Receptacle_USB2.0
- removed R2: 0, symbol Device:R_US
- added J3: 105450-0101, USB Receptale:MOLEX_105450-0101, symbol USB_TYPE_C:105450-0101
- C1, C2, C3, C4, C5, C6, C7, C8: footprint (none) -> Capacitor_SMD:C_0603_1608Metric
- F1: footprint (none) -> Fuse:Fuse_0805_2012Metric
- J1: footprint (none) -> Connector_PinHeader_2.54mm:PinHeader_1x01_P2.54mm_Vertical
- J10: renamed from J8; footprint (none) -> Connector_PinHeader_2.54mm:PinHeader_2x05_P2.54mm_Vertical
- J11: renamed from J9; footprint (none) -> Connector_PinHeader_2.54mm:PinHeader_1x08_P2.54mm_Vertical
- J2: footprint (none) -> Connector_PinHeader_2.54mm:PinHeader_1x06_P2.54mm_Vertical
- J4: renamed from J?; value Conn_01x06_Female -> I/O_TEST; footprint (none) -> Connector_PinHeader_2.54mm:PinHeader_1x06_P2.54mm_Vertical
- J5: renamed from J?; value Conn_01x04_Female -> GND_test; footprint (none) -> Connector_PinHeader_2.54mm:PinHeader_1x04_P2.54mm_Vertical
- J6: renamed from J4; footprint (none) -> Connector_PinHeader_2.54mm:PinHeader_1x08_P2.54mm_Vertical
- J7: renamed from J5; footprint (none) -> Connector_PinHeader_2.54mm:PinHeader_1x01_P2.54mm_Vertical
- J8: renamed from J6; footprint (none) -> Connector_PinHeader_2.54mm:PinHeader_1x10_P2.54mm_Vertical
- J9: renamed from J7; footprint (none) -> Connector_PinHeader_2.54mm:PinHeader_1x06_P2.54mm_Vertical
- R1, R3: footprint (none) -> Resistor_SMD:R_0603_1608Metric
- R2: renamed from R4; footprint (none) -> Resistor_SMD:R_0603_1608Metric
- R4: renamed from R5; footprint (none) -> Resistor_SMD:R_0603_1608Metric
- R5: renamed from R6; footprint (none) -> Resistor_SMD:R_0603_1608Metric
- TP1, TP2, TP3, TP4, TP5, TP6: footprint (none) -> TestPoint:TestPoint_Pad_4.0x4.0mm
- U2: footprint PW20 -> TXB108:TXB0108PWR
- U3: footprint Package_TO_SOT_THT:TO-3 -> Package_TO_SOT_THT:TO-220-3_Vertical
Connections:
- net GND: now also J3.A1 (GND1), J3.A12 (GND2), J3.B1 (GND3), J3.B12 (GND4), J3.S1 (SHIELD), J3.S2 (SHIELD), J3.S3 (SHIELD), J3.S4 (SHIELD)
- net at F1.1: now also J3.A4 (VBUS1), J3.A9 (VBUS2), J3.B4 (VBUS3), J3.B9 (VBUS4)
- net at R2.1: now also J3.A5 (CC1)
- net at R3.1: now also J3.B5 (CC2)
- new net: J3.A6 (D1+), J3.A7 (D1-)
- new net: J3.B6 (D2+), J3.B7 (D2-)
Other:
- moved on the sheet: J11, R2, R3

Commit message: PCB first board ready/Debugging UART
Parts:
- added C10, C9: 20pf, Capacitor_SMD:C_0603_1608Metric, symbol Device:C
- added C11: 1n, Capacitor_SMD:C_0603_1608Metric, symbol Device:C
- added R10, R11, R12, R16, R6, R7, R8, R9: 5k, Resistor_SMD:R_0603_1608Metric, symbol Device:R_US
- added R13, R14: 0, Resistor_SMD:R_0603_1608Metric, symbol Device:R_US
- added R15: 1M, Resistor_SMD:R_0603_1608Metric, symbol Device:R_US
- added SW1: EN, Button_Switch_THT:SW_PUSH_6mm, symbol Switch:SW_Push
- added SW2: ID0, Button_Switch_THT:SW_PUSH_6mm, symbol Switch:SW_Push
- added Y1: ECS-160-20-3X-TR, 16 MHz Crystal:XTAL_ECS-160-20-3X-TR, symbol 16_MHz_Crystal:ECS-160-20-3X-TR
- TP1, TP4: value TestPoint_Flag -> TEST_TX; footprint TestPoint:TestPoint_Pad_4.0x4.0mm -> Connector_PinHeader_2.54mm:PinHeader_1x01_P2.54mm_Vertical
- TP2: footprint TestPoint:TestPoint_Pad_4.0x4.0mm -> Connector_PinHeader_2.54mm:PinHeader_1x01_P2.54mm_Vertical
- TP3: value TestPoint_Flag -> TEST_RX; footprint TestPoint:TestPoint_Pad_4.0x4.0mm -> Connector_PinHeader_2.54mm:PinHeader_1x01_P2.54mm_Vertical
- TP5: value TestPoint_Flag -> TEST_5V; footprint TestPoint:TestPoint_Pad_4.0x4.0mm -> Connector_PinHeader_2.54mm:PinHeader_1x01_P2.54mm_Vertical
- TP6: value TestPoint_Flag -> TEST_3.3V; footprint TestPoint:TestPoint_Pad_4.0x4.0mm -> Connector_PinHeader_2.54mm:PinHeader_1x01_P2.54mm_Vertical
Connections:
- net I034 is gone; now on net IO34: J4.2 (Pin_2)
- net IO32 is gone; now on net I032: J4.4 (Pin_4)
- net IO33 is gone; now on net I033: J4.5 (Pin_5)
- net +3V3: now also R13.1, R6.1, R7.1
- net +5V: now also R10.1, R11.1, R12.1, R8.1, R9.1
- net GND: now also U2.11 (GND), C10.2, C11.1, C9.2, R14.2, R16.2, SW1.1, SW2.1
- net PC0: now reaches J9.1 (Pin_1), U4.23 (PC0)
- net PC1: now reaches J9.2 (Pin_2), U4.24 (PC1)
- net PC2: now reaches J9.3 (Pin_3), U4.25 (PC2)
- net PC3: now reaches J9.4 (Pin_4), U4.26 (PC3)
- net at J6.1 (Pin_1), TP3.1, U2.18 (B2)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: now also R8.2
- net at J6.2 (Pin_2), TP4.1, U2.17 (B3)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: now also R9.2
- net PD2: now reaches J6.3 (Pin_3), U4.32 (PD2)
- net PD3: now reaches J6.4 (Pin_4), U4.1 (PD3)
- net PD4: now reaches J6.5 (Pin_5), U4.2 (PD4)
- net PD5: now reaches J6.6 (Pin_6), U4.9 (PD5)
- net PD6: now reaches J6.7 (Pin_7), U4.10 (PD6)
- net PD7: now reaches J6.8 (Pin_8), U4.11 (PD7)
- net PB0: now reaches J8.1 (Pin_1), U4.12 (PB0)
- net PB1: now reaches J8.2 (Pin_2), U4.13 (PB1)
- net PB2: now reaches J8.3 (Pin_3), U4.14 (PB2)
- net at J10.1 (MOSI), J8.4 (Pin_4), U4.15 (PB3): now also R11.2
- net at J10.9 (MISO), J8.5 (Pin_5), U4.16 (PB4): now also R12.2
- net at J10.7 (SCK), J8.6 (Pin_6), U4.17 (PB5): now also R10.2
- net at U1.24 (IO2): now also R16.1
- net IO0: now reaches J4.1 (Pin_1), U1.25 (IO0)
- net IO0: now also C11.2, SW2.2
- net at C1.1, R1.1, U1.3 (EN): now also SW1.2
- net at J2.2 (Pin_2), TP2.1, U1.34 (RXD0)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: now also R7.2
- net at J2.3 (Pin_3), TP1.1, U1.35 (TXD0)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: now also R6.2
- net OE: now reaches U2.10 (OE)
- net OE: now also R13.2, R14.1
- net PB6: now reaches U4.7 (PB6)
- net PB6: now also C10.1, R15.2, Y1.2
- net PB7: now reaches U4.8 (PB7)
- net PB7: now also C9.1, R15.1, Y1.1
- no-connect marks 0 -> 52
Other:
- moved on the sheet: C2, C5, J1, R1, TP1, TP2, TP3, TP4
